File: ASIC3_PCB/ASIC3_PCB.kicad_pcb (KiCad board)
At the start: 6 copper layers, 36.5 x 30.4 mm, 44 parts, among them J100 MOLEX-524653071, J11 MEC5-040-01-L-RA-W2-TR, J200 MOLEX-524653071, J3 Connector, J6 MOLEX-524653071, J7 MOLEX-524653071, J99 5024262030, U1 ASIC3_M

Commit message: remove bottom connector to second ASIC
Parts:
- removed J100, J7: MOLEX-524653071, FDM_footprints:J524653071_Board2Board
Connections:
- U1 pad 109: unconnected-(U1-109_GND-Pad109) -> /SER_CLK_0
Routing:
- net /SER_CLK_0: track 0.00 -> 4.06 mm
- net (no net): track 4.06 -> 0.00 mm
