File: ASIC3_PCB/ASIC3_PCB.kicad_sch (KiCad schematic)
At the start: 44 parts, among them J100 MOLEX-524653071, J11 MEC5-040-01-L-RA-W2-TR, J200 MOLEX-524653071, J3 Connector, J6 MOLEX-524653071, J7 MOLEX-524653071, J99 5024262030, U1 ASIC3_M

Commit message: remove bottom connector to second ASIC
Parts:
- removed J100, J7: MOLEX-524653071, FDM_footprints:J524653071_Board2Board, symbol FDM_project_Library:Board2Board_MOLEX-5009130302_1
Other:
- note removed: "${##}"
- note removed: "${#}"
- note removed: "${CURRENT_DATE}"
- note removed: "${DOCUMENTFULLPATHANDNAME}"
- note removed: "${REVISION}"
- note removed: "${SHEET}"
- note removed: "${TITLE}"
- note removed: "72770 Reutlingen"
- note removed: "Aspenhaustrasse 21"
- note removed: "CJ/"
- note removed: "Germany"
- note removed: "Multi Channel Systems MCS GmbH"
- note removed: "date:"
- note removed: "drawn by: RM"
- note removed: "file:"
- note removed: "of"
- note removed: "revision:"
- note removed: "sheet"
- note removed: "size: A4"
- title: BrainCom ASIC2 Level -> BrainCom ASIC3 Level
